File: pcb/panel.kicad_pcb (KiCad board)
At the start: 2 copper layers, 181 x 99.1 mm, 107 parts, among them P1 CONN_01X09, SW1 SWITCH_INV, SW10 SWITCH_INV, SW11 SWITCH_INV, SW12 SWITCH_INV, SW13 SWITCH_INV, SW14 SWITCH_INV, SW15 SWITCH_INV, SW16 SWITCH_INV, SW17 SP3T, SW18 SP3T, SW19 SP3T, SW2 SWITCH_INV, SW20 SP3T, SW3 SWITCH_INV, SW4 SWITCH_INV, SW5 SWITCH_INV, SW6 SWITCH_INV, SW7 SWITCH_INV, SW8 SWITCH_INV, SW9 SWITCH_INV, U1 74HC595, U2 74HC595, U3 74HC595, U4 74HC595, U5 23LC1024, U6 74LS165, U7 74LS165, U8 74LS165, U9 CONN_microSD

Commit message: Changed value of R33 to 220 Ohms. New value found through testing.
Parts:
- R33: value 10K -> 220R
